File: BRUTUS CONTROL BOARD.brd (EAGLE design)
At the start: 110.5 x 86.4 mm, 42 parts, among them IC1 74LS14N, IC2 74LS595N, IC3 74LS595N, IC5 4021N, IC6 4021N, Q1 16MHz, X1 5566-6, X2 5566-16, X3 5566-2, X4 5566-4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

Commit message: 4th commit
Changed lines of the file:
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@@
 <text x="6.35" y="39.37" size="1.778" layer="112">OUT</text>
 <text x="35.56" y="3.81" size="1.778" layer="112">IN</text>
-<text x="8.89" y="80.01" size="1.778" layer="112">BREWERY CONTROLLER
+<text x="15.24" y="80.01" size="1.778" layer="112">BREWERY CONTROLLER
 K. NILSSON 2015-06-27</text>
 </plain>
