File: RTD COMPARATOR BOARD.sch (EAGLE design)
At the start: 50 parts, among them IC1 LM324N, IC2 LM324N, IC3 LM324N, IC4 LM324N, IC5 LM324N, IC6 LM324N, IC7 LM324N, IC8 LM324N, IC9 LM324N, X1 5566-10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

Commit message: 4th commit
Parts:
- removed IC4, IC5, IC6, IC7, IC8, IC9: LM324N, linear:LM324N
- R22, R23, R24: value 1k -> 10k
- R34: value 220 -> 220k
Connections:
- new net N$11: R23.1, X1-7.S
- new net N$3: R24.1, X1-1.S
- net N$10: now also IC2A.+IN; no longer IC4A.+IN
- net N$14: no longer R22.1
- net N$15: now also IC2A.-IN, IC2A.OUT; no longer IC4A.-IN, IC4A.OUT, IC4P.V-
- net N$16: now also IC2C.-IN; no longer IC6A.-IN
- net N$18: now also IC1C.-IN; no longer IC3A.-IN
- net N$19: no longer IC1P.V-
- net N$20: now also IC2B.-IN, IC2B.OUT; no longer IC5A.-IN, IC5A.OUT, IC5P.V-
- net N$21: now also IC1B.-IN, IC1B.OUT; no longer IC2A.-IN, IC2A.OUT, IC2P.V-
- net N$22: now also IC1C.+IN; no longer IC3A.+IN
- net N$23: now also IC1C.OUT; no longer IC3A.OUT
- net N$24: now also C3.1, IC1B.+IN, X1-2.S; no longer IC2A.+IN
- net N$25: no longer C2.1, R23.1
- net N$26: now also IC2C.+IN; no longer IC6A.+IN
- net N$29: now also IC2C.OUT; no longer IC6A.OUT
- net N$32: now also IC3B.+IN; no longer IC8A.+IN
- net N$33: now also IC3A.+IN; no longer IC7A.+IN
- net N$34: now also IC3A.-IN, IC3A.OUT; no longer IC7A.-IN, IC7A.OUT, IC7P.V-
- net N$35: now also IC3C.-IN; no longer IC9A.-IN
- net N$36: now also IC3B.-IN, IC3B.OUT; no longer IC8A.-IN, IC8A.OUT, IC8P.V-
- net N$37: now also IC3C.+IN; no longer IC9A.+IN
- net N$38: now also IC3C.OUT; no longer IC9A.OUT
- net N$4: now also R22.1, X1-4.S; no longer C3.1, R24.1, X1-2.S
- net N$9: now also IC2B.+IN; no longer IC5A.+IN
- net VCC: no longer X1-1.S, X1-4.S, X1-7.S
Other:
- moved on the sheet: IC2A, IC3A, R22, R23, R24, X1-8
